Commit message: master

File: ros/src/car_model/urdf/smart.xacro (robot description, xacro)
@@ -4,12 +4,12 @@
   <xacro:property name="PI" value="3.1415926835897931"/>
   <!-- base -->
-  <xacro:property name="base_length" value="2.695"/>
+  <xacro:property name="base_length" value="3.8"/>
   <xacro:property name="base_width" value="0.68"/>
   <xacro:property name="base_height" value="1.370"/>
   <xacro:property name="base_collision_height" value="0.875"/>
-  <xacro:property name="base_mass" value="956"/>
+  <xacro:property name="base_mass" value="2080"/>
   <xacro:property name="base_mass_ixx" value="343"/>
   <xacro:property name="base_mass_iyy" value="728"/>
-  <xacro:property name="base_mass_izz" value="772"/>
+  <xacro:property name="base_mass_izz" value="7508.800"/>
   <!-- rear tyre -->
   <xacro:property name="rear_tyre_x" value="0.945"/>
